Commit message: Gazebo simulation works

File: bittle_description/xacro/bittle.urdf.xacro (robot description, xacro)
@@ -15,9 +15,13 @@
     <xacro:leg hside="right" vside="front">
         <origin xyz="0.45149 0.52264 -0.02102" rpy="-1.5708 0 -1.5708"/>
-        <origin xyz="0.00006 0.49938 0.03996" rpy="0 0 3.14159"/>
+        <origin xyz="0.00006 0.49938 0.03996" rpy="0. 0. ${pi}"/>
     </xacro:leg>
     <xacro:leg hside="right" vside="back">
         <origin xyz="0.45149 -0.51923 -0.02102" rpy="-1.5708 0 -1.5708"/>
-        <origin xyz="0.00015 0.49938 0.03996" rpy="0 0 3.14159"/>
+        <origin xyz="0.00015 0.49938 0.03996" rpy="0. 0. ${pi}"/>
     </xacro:leg>
+    <!-- Joint states plugin -->
+    <gazebo>
+        <plugin filename="ignition-gazebo-joint-state-publisher-system" name="ignition::gazebo::systems::JointStatePublisher"/>
+    </gazebo>
 </robot>

File: bittle_description/xacro/bittle/leg.urdf.xacro (robot description, xacro)
@@ -1,87 +1,126 @@
 <?xml version="1.0"?>
 <robot xmlns:xacro="http://www.ros.org/wiki/xacro">
-    <xacro:macro name="leg" params="hside vside
-        *origin_shoulder
-        *origin_knee">
-        <joint name="${hside}_${vside}_shoulder_joint" type="revolute">
-            <xacro:insert_block name="origin_shoulder"/>
-            <parent link="base_frame_link"/>
-            <child link="${hside}_${vside}_shoulder_link"/>
-            <axis xyz="0 0 1"/>
-            <limit lower="-1.5708" upper="1.22173" effort="1.0" velocity="1.5708"/>
-        </joint>
-        <link name="${hside}_${vside}_shoulder_link">
-            <visual>
-                <xacro:if value="${hside == 'left'}">
-                    <origin xyz="0 -0.24575 0.0777" rpy="-1.5708 1.5708 -1.5708"/>
-                </xacro:if>
-                <xacro:if value="${hside == 'right'}">
-                    <origin xyz="0 0.24575 0.0777" rpy="1.5708 -1.5708 -1.5708"/>
-                </xacro:if>
-                <geometry>
-                    <mesh filename="package://bittle_description/meshes/visual/shoulder.stl"/>
-                </geometry>
-                <material name="yellow"/>
-            </visual>
-            <collision>
-                <xacro:if value="${hside == 'left'}">
-                    <origin xyz="0 -0.24575 0.0777" rpy="-1.5708 1.5708 -1.5708"/>
-                </xacro:if>
-                <xacro:if value="${hside == 'right'}">
-                    <origin xyz="0 0.24575 0.0777" rpy="1.5708 -1.5708 -1.5708"/>
-                </xacro:if>
-                <geometry>
-                    <mesh filename="package://bittle_description/meshes/visual/shoulder.stl"/>
-                </geometry>
-            </collision>
-            <inertial>
-                <origin xyz="0 -0.24575 0.04372" rpy="0 0 0"/>
-                <mass value="0.006"/>
-                <inertia
-                    ixx="0.00044" ixy="0" ixz="0"
-                    iyy="0.00005" iyz="0"
-                    izz="0.00044" />
-            </inertial>
-        </link>
-        <joint name="${hside}_${vside}_knee_joint" type="revolute">
-            <xacro:insert_block name="origin_knee"/>
-            <parent link="${hside}_${vside}_shoulder_link"/>
-            <child link="${hside}_${vside}_knee_link"/>
-            <axis xyz="0 0 1"/>
-            <limit lower="-1.22173" upper="1.48353" effort="1.0" velocity="1.5708"/>
-        </joint>
-        <link name="${hside}_${vside}_knee_link">
-            <visual>
-                <xacro:if value="${hside == 'left'}">
-                    <origin xyz="-0.09232 0 -0.14614" rpy="-1.5708 1.5708 0"/>
-                </xacro:if>
-                <xacro:if value="${hside == 'right'}">
-                    <origin xyz="0.09497 -0.00238 -0.1382" rpy="-1.5708 -1.5708 0"/>
-                </xacro:if>
-                <geometry>
-                    <mesh filename="package://bittle_description/meshes/visual/${hside}_knee.stl"/>
-                </geometry>
-                <material name="black"/>
-            </visual>
-            <collision>
-                <xacro:if value="${hside == 'left'}">
-                    <origin xyz="-0.09232 0 -0.14614" rpy="-1.5708 1.5708 0"/>
-                </xacro:if>
-                <xacro:if value="${hside == 'right'}">
-                    <origin xyz="0.09497 -0.00238 -0.1382" rpy="-1.5708 -1.5708 0"/>
-                </xacro:if>
-                <geometry>
-                    <mesh filename="package://bittle_description/meshes/visual/${hside}_knee.stl"/>
-                </geometry>
-            </collision>
-            <inertial>
-                <origin xyz="-0.08998 0 -0.14638" rpy="0 0 0"/>
-                <mass value="0.017"/>
-                <inertia
-                    ixx="0.00006" ixy="0" ixz="0"
-                    iyy="0.00065" iyz="0"
-                    izz="0.00063" />
-            </inertial>
-        </link>
-    </xacro:macro>
+  <xacro:macro name="leg" params="hside vside
+    *origin_shoulder
+    *origin_knee">
+    <joint name="${hside}_${vside}_shoulder_joint" type="revolute">
+      <xacro:insert_block name="origin_shoulder"/>
+      <parent link="base_frame_link"/>
+      <child link="${hside}_${vside}_shoulder_link"/>
+      <xacro:if value="${hside == 'left'}">
+        <axis xyz="0 0 1"/>
+      </xacro:if>
+      <xacro:if value="${hside == 'right'}">
+        <axis xyz="0 0 -1"/>
+      </xacro:if>
+      <limit lower="-1.5708" upper="1.22173" effort="1.0" velocity="1.5708"/>
+    </joint>
+    <!-- Joint controller plugin -->
+    <!--
+    <gazebo>
+      <plugin filename="ignition-gazebo-joint-controller-system"
+            name="ignition::gazebo::systems::JointController">
+        <joint_name>${hside}_${vside}_shoulder_joint</joint_name>
+      </plugin>
+    </gazebo>
+    -->
+    <gazebo>
+      <plugin filename="ignition-gazebo-joint-position-controller-system"
+              name="ignition::gazebo::systems::JointPositionController">
+        <joint_name>${hside}_${vside}_shoulder_joint</joint_name>
+        <topic>/joint/${hside}_${vside}_shoulder_joint/cmd_pos</topic>
+      </plugin>
+    </gazebo>
+    <link name="${hside}_${vside}_shoulder_link">
+      <visual>
+        <xacro:if value="${hside == 'left'}">
+          <origin xyz="0 -0.24575 0.0777" rpy="-1.5708 1.5708 -1.5708"/>
+        </xacro:if>
+        <xacro:if value="${hside == 'right'}">
+          <origin xyz="0 0.24575 0.0777" rpy="1.5708 -1.5708 -1.5708"/>
+        </xacro:if>
+        <geometry>
+          <mesh filename="package://bittle_description/meshes/visual/shoulder.stl"/>
+        </geometry>
+        <material name="yellow"/>
+      </visual>
+      <collision>
+        <xacro:if value="${hside == 'left'}">
+          <origin xyz="0 -0.24575 0.0777" rpy="-1.5708 1.5708 -1.5708"/>
+        </xacro:if>
+        <xacro:if value="${hside == 'right'}">
+          <origin xyz="0 0.24575 0.0777" rpy="1.5708 -1.5708 -1.5708"/>
+        </xacro:if>
+        <geometry>
+          <mesh filename="package://bittle_description/meshes/visual/shoulder.stl"/>
+        </geometry>
+      </collision>
+      <inertial>
+        <origin xyz="0 -0.24575 0.04372" rpy="0 0 0"/>
+        <mass value="0.006"/>
+        <inertia
+            ixx="0.00044" ixy="0" ixz="0"
+            iyy="0.00005" iyz="0"
+            izz="0.00044" />
+      </inertial>
+    </link>
+    <joint name="${hside}_${vside}_knee_joint" type="revolute">
+      <xacro:insert_block name="origin_knee"/>
+      <parent link="${hside}_${vside}_shoulder_link"/>
+      <child link="${hside}_${vside}_knee_link"/>
+      <xacro:if value="${hside == 'left'}">
+        <axis xyz="0 0 1"/>
+      </xacro:if>
+      <xacro:if value="${hside == 'right'}">
+        <axis xyz="0 0 -1"/>
+      </xacro:if>
+      <limit lower="-1.22173" upper="1.48353" effort="1.0" velocity="1.5708"/>
+    </joint>
+    <!-- Joint controller plugin -->
+    <!-- <gazebo>
+      <plugin filename="ignition-gazebo-joint-controller-system" name="ignition::gazebo::systems::JointController">
+          <joint_name>${hside}_${vside}_knee_joint</joint_name>
+      </plugin>
+    </gazebo> -->
+    <gazebo>
+      <plugin filename="ignition-gazebo-joint-position-controller-system"
+              name="ignition::gazebo::systems::JointPositionController">
+        <joint_name>${hside}_${vside}_knee_joint</joint_name>
+        <topic>/joint/${hside}_${vside}_knee_joint/cmd_pos</topic>
+      </plugin>
+    </gazebo>
+    <link name="${hside}_${vside}_knee_link">
+      <visual>
+        <xacro:if value="${hside == 'left'}">
+          <origin xyz="-0.09232 0 -0.14614" rpy="-1.5708 1.5708 0"/>
+        </xacro:if>
+        <xacro:if value="${hside == 'right'}">
+          <origin xyz="0.09497 -0.00238 -0.1382" rpy="-1.5708 -1.5708 0"/>
+        </xacro:if>
+        <geometry>
+          <mesh filename="package://bittle_description/meshes/visual/${hside}_knee.stl"/>
+        </geometry>
+        <material name="black"/>
+      </visual>
+      <collision>
+        <xacro:if value="${hside == 'left'}">
+          <origin xyz="-0.09232 0 -0.14614" rpy="-1.5708 1.5708 0"/>
+        </xacro:if>
+        <xacro:if value="${hside == 'right'}">
+          <origin xyz="0.09497 -0.00238 -0.1382" rpy="-1.5708 -1.5708 0"/>
+        </xacro:if>
+        <geometry>
+          <mesh filename="package://bittle_description/meshes/visual/${hside}_knee.stl"/>
+        </geometry>
+      </collision>
+      <inertial>
+        <origin xyz="-0.08998 0 -0.14638" rpy="0 0 0"/>
+        <mass value="0.017"/>
+        <inertia
+            ixx="0.00006" ixy="0" ixz="0"
+            iyy="0.00065" iyz="0"
+            izz="0.00063" />
+      </inertial>
+    </link>
+  </xacro:macro>
 </robot>

File: bittle_description/xacro/bittle/mainboard.urdf.xacro (robot description, xacro)
@@ -1,49 +1,61 @@
 <?xml version="1.0"?>
 <robot xmlns:xacro="http://www.ros.org/wiki/xacro">
-    <xacro:macro name="mainboard" params="prefix:=''">
-        <joint name="mainboard_joint" type="fixed">
-            <origin xyz="0.00652 -0.00827 0.06423" rpy="0 0 0"/>
-            <parent link="base_frame_link"/>
-            <child link="mainboard_link"/>
-        </joint>
-        <link name="mainboard_link">
-            <visual>
-                <origin xyz="0 0 0" rpy="0 0 0"/>
-                <geometry>
-                    <mesh filename="package://bittle_description/meshes/visual/plane.stl"/>
-                </geometry>
-                <material name="alluminium"/>
-            </visual>
-            <inertial>
-                <origin xyz="0 0 0" rpy="0 0 0"/>
-                <mass value="0.001"/>
-                <inertia
-                    ixx="0.001" ixy="0" ixz="0"
-                    iyy="0.001" iyz="0"
-                    izz="0.001" />
-            </inertial>
-        </link>
-        <joint name="imu_joint" type="fixed">
-            <origin xyz="-0.00652 0.00827 0.00586" rpy="0 0 -3.14159"/>
-            <parent link="mainboard_link"/>
-            <child link="imu_link"/>
-        </joint>
-        <link name="imu_link">
-            <visual>
-                <origin xyz="0 0 0" rpy="0 0 3.14159"/>
-                <geometry>
-                    <mesh filename="package://bittle_description/meshes/visual/imu.stl"/>
-                </geometry>
-                <material name="black"/>
-            </visual>
-            <inertial>
-                <origin xyz="0 0 0" rpy="0 0 0"/>
-                <mass value="0.001"/>
-                <inertia
-                    ixx="0.001" ixy="0" ixz="0"
-                    iyy="0.001" iyz="0"
-                    izz="0.001" />
-            </inertial>
-        </link>
-    </xacro:macro>
+  <xacro:macro name="mainboard" params="prefix:=''">
+    <joint name="mainboard_joint" type="fixed">
+      <origin xyz="0.00652 -0.00827 0.06423" rpy="0 0 0"/>
+      <parent link="base_frame_link"/>
+      <child link="mainboard_link"/>
+    </joint>
+    <link name="mainboard_link">
+      <visual>
+        <origin xyz="0 0 0" rpy="0 0 0"/>
+        <geometry>
+          <mesh filename="package://bittle_description/meshes/visual/plane.stl"/>
+        </geometry>
+        <material name="alluminium"/>
+      </visual>
+      <inertial>
+        <origin xyz="0 0 0" rpy="0 0 0"/>
+        <mass value="0.001"/>
+        <inertia
+          ixx="0.001" ixy="0" ixz="0"
+          iyy="0.001" iyz="0"
+          izz="0.001" />
+      </inertial>
+    </link>
+    <joint name="imu_joint" type="fixed">
+      <origin xyz="-0.00652 0.00827 0.00586" rpy="0. 0. ${-pi}"/>
+      <parent link="mainboard_link"/>
+      <child link="imu_link"/>
+    </joint>
+    <link name="imu_link">
+      <visual>
+        <origin xyz="0 0 0" rpy="0. 0. ${pi}"/>
+        <geometry>
+          <mesh filename="package://bittle_description/meshes/visual/imu.stl"/>
+        </geometry>
+        <material name="black"/>
+      </visual>
+      <inertial>
+        <origin xyz="0 0 0" rpy="0 0 0"/>
+        <mass value="0.001"/>
+        <inertia
+          ixx="0.001" ixy="0" ixz="0"
+          iyy="0.001" iyz="0"
+          izz="0.001" />
+      </inertial>
+      <gazebo>
+        <sensor name="imu_sensor" type="imu">
+          <always_on>1</always_on>
+          <update_rate>10</update_rate>
+          <visualize>true</visualize>
+          <topic>imu</topic>
+        </sensor>
+      </gazebo>
+    </link>
+    <!-- Imu plugin -->
+    <gazebo>
+      <plugin filename="ignition-gazebo-imu-system" name="ignition::gazebo::systems::Imu"/>
+    </gazebo>
+  </xacro:macro>
 </robot>
